File: kicad/atmega328p.kicad_sch (KiCad schematic)
At the start: 10 parts, among them Q1 PMOS - LP0701N3-G, SW1 SW_Push, U1 ATmega328-P, Y1 16Mhz

Commit message: Updated board schematic and layout because of FET labeled incorrectly in schematic.
Connections:
- net VCC: now also Q1.3 (S); no longer Q1.1 (D)
- net VREF: now also Q1.1 (D); no longer Q1.3 (S)
Changed lines of the file:
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@@
 (kicad_sch (version 20230121) (generator eeschema)
-  (paper "A4")
+  (paper "USLegal")
   (title_block
     (title "Arduino Waveshare 7.3F e-paper Dislay")
-    (date "2023-04-14")
-    (rev "V01")
+    (date "2024-01-08")
+    (rev "V02")
     (comment 2 "creativecommons.org/licenses/by/4.0")
     (comment 3 "License: CC BY 4.0")
@@
     (instances
       (project "epaper_board_layout"
-        (path "/e3b1e824-2fe0-40f4-81c0-a3915952426b"
+        (path "/e3b1e824-2fe0-40f4-81c0-a3915952426b/d4ff5ade-77fa-490a-a921-760304d03ec6"
           (reference "C1") (unit 1)
         )
-        (path "/e3b1e824-2fe0-40f4-81c0-a3915952426b/9d2591fc-d2e2-4b8a-a8a8-120035ff8a59"
-          (reference "C1") (unit 1)
-        )
-        (path "/e3b1e824-2fe0-40f4-81c0-a3915952426b/d4ff5ade-77fa-490a-a921-760304d03ec6"
-          (reference "C1") (unit 1)
-        )
       )
     )
@@
   (symbol (lib_id "power:GND") (at 95.25 129.54 0) (unit 1)
     (in_bom yes) (on_board yes) (dnp no) (fields_autoplaced)
-    (property "Reference" "#PWR01" (at 95.25 135.89 0)
+    (property "Reference" "#PWR02" (at 95.25 135.89 0)
       (effects (font (size 1.27 1.27)) hide)
     )
@@
     (instances
       (project "epaper_board_layout"
-        (path "/e3b1e824-2fe0-40f4-81c0-a3915952426b"
-          (reference "#PWR01") (unit 1)
-        )
-        (path "/e3b1e824-2fe0-40f4-81c0-a3915952426b/9d2591fc-d2e2-4b8a-a8a8-120035ff8a59"
+        (path "/e3b1e824-2fe0-40f4-81c0-a3915952426b/d4ff5ade-77fa-490a-a921-760304d03ec6"
           (reference "#PWR02") (unit 1)
         )
-        (path "/e3b1e824-2fe0-40f4-81c0-a3915952426b/d4ff5ade-77fa-490a-a921-760304d03ec6"
-          (reference "#PWR02") (unit 1)
-        )
-      )
-    )
-  )
-  (symbol (lib_id "Simulation_SPICE:PMOS") (at 226.06 130.81 0) (unit 1)
-    (in_bom yes) (on_board yes) (dnp no) (fields_autoplaced)
-    (property "Reference" "Q1" (at 232.41 130.175 0)
+      )
+    )
+  )
+  (symbol (lib_id "Simulation_SPICE:PMOS") (at 226.06 130.81 0) (mirror x) (unit 1)
+    (in_bom yes) (on_board yes) (dnp no)
+    (property "Reference" "Q1" (at 232.41 131.445 0)
       (effects (font (size 1.27 1.27)) (justify left))
     )
-    (property "Value" "PMOS - LP0701N3-G" (at 232.41 132.715 0)
+    (property "Value" "PMOS - LP0701N3-G" (at 232.41 128.905 0)
       (effects (font (size 1.27 1.27)) (justify left))
     )
-    (property "Footprint" "Package_TO_SOT_THT:TO-92" (at 231.14 128.27 0)
-      (effects (font (size 1.27 1.27)) hide)
-    )
-    (property "Datasheet" "https://www.digikey.com/en/products/detail/microchip-technology/lp0701n3-g/4902364" (at 226.06 143.51 0)
-      (effects (font (size 1.27 1.27)) hide)
-    )
-    (property "Sim.Device" "PMOS" (at 226.06 147.955 0)
-      (effects (font (size 1.27 1.27)) hide)
-    )
-    (property "Sim.Type" "VDMOS" (at 226.06 149.86 0)
-      (effects (font (size 1.27 1.27)) hide)
-    )
-    (property "Sim.Pins" "1=D 2=G 3=S" (at 226.06 146.05 0)
+    (property "Footprint" "Package_TO_SOT_THT:TO-92" (at 231.14 133.35 0)
+      (effects (font (size 1.27 1.27)) hide)
+    )
+    (property "Datasheet" "https://www.digikey.com/en/products/detail/microchip-technology/lp0701n3-g/4902364" (at 226.06 118.11 0)
+      (effects (font (size 1.27 1.27)) hide)
+    )
+    (property "Sim.Device" "PMOS" (at 226.06 113.665 0)
+      (effects (font (size 1.27 1.27)) hide)
+    )
+    (property "Sim.Type" "VDMOS" (at 226.06 111.76 0)
+      (effects (font (size 1.27 1.27)) hide)
+    )
+    (property "Sim.Pins" "1=S 2=G 3=D" (at 226.06 115.57 0)
       (effects (font (size 1.27 1.27)) hide)
     )
@@
     (instances
       (project "epaper_board_layout"
-        (path "/e3b1e824-2fe0-40f4-81c0-a3915952426b"
-          (reference "#PWR03") (unit 1)
-        )
-        (path "/e3b1e824-2fe0-40f4-81c0-a3915952426b/9d2591fc-d2e2-4b8a-a8a8-120035ff8a59"
-          (reference "#PWR03") (unit 1)
-        )
         (path "/e3b1e824-2fe0-40f4-81c0-a3915952426b/d4ff5ade-77fa-490a-a921-760304d03ec6"
           (reference "#PWR03") (unit 1)
@@
     (instances
       (project "epaper_board_layout"
-        (path "/e3b1e824-2fe0-40f4-81c0-a3915952426b"
+        (path "/e3b1e824-2fe0-40f4-81c0-a3915952426b/d4ff5ade-77fa-490a-a921-760304d03ec6"
           (reference "U1") (unit 1)
         )
-        (path "/e3b1e824-2fe0-40f4-81c0-a3915952426b/9d2591fc-d2e2-4b8a-a8a8-120035ff8a59"
-          (reference "U1") (unit 1)
-        )
-        (path "/e3b1e824-2fe0-40f4-81c0-a3915952426b/d4ff5ade-77fa-490a-a921-760304d03ec6"
-          (reference "U1") (unit 1)
-        )
       )
     )
@@
     (instances
       (project "epaper_board_layout"
-        (path "/e3b1e824-2fe0-40f4-81c0-a3915952426b"
-          (reference "C2") (unit 1)
-        )
-        (path "/e3b1e824-2fe0-40f4-81c0-a3915952426b/9d2591fc-d2e2-4b8a-a8a8-120035ff8a59"
-          (reference "C2") (unit 1)
-        )
         (path "/e3b1e824-2fe0-40f4-81c0-a3915952426b/d4ff5ade-77fa-490a-a921-760304d03ec6"
           (reference "C2") (unit 1)
@@
     (instances
       (project "epaper_board_layout"
-        (path "/e3b1e824-2fe0-40f4-81c0-a3915952426b"
+        (path "/e3b1e824-2fe0-40f4-81c0-a3915952426b/d4ff5ade-77fa-490a-a921-760304d03ec6"
           (reference "Y1") (unit 1)
         )
-        (path "/e3b1e824-2fe0-40f4-81c0-a3915952426b/9d2591fc-d2e2-4b8a-a8a8-120035ff8a59"
-          (reference "Y1") (unit 1)
-        )
-        (path "/e3b1e824-2fe0-40f4-81c0-a3915952426b/d4ff5ade-77fa-490a-a921-760304d03ec6"
-          (reference "Y1") (unit 1)
-        )
       )
     )
@@
   (symbol (lib_id "power:VCC") (at 95.25 43.18 0) (unit 1)
     (in_bom yes) (on_board yes) (dnp no) (fields_autoplaced)
-    (property "Reference" "#PWR02" (at 95.25 46.99 0)
+    (property "Reference" "#PWR01" (at 95.25 46.99 0)
       (effects (font (size 1.27 1.27)) hide)
     )
@@
     (instances
       (project "epaper_board_layout"
-        (path "/e3b1e824-2fe0-40f4-81c0-a3915952426b"
-          (reference "#PWR02") (unit 1)
-        )
-        (path "/e3b1e824-2fe0-40f4-81c0-a3915952426b/9d2591fc-d2e2-4b8a-a8a8-120035ff8a59"
+        (path "/e3b1e824-2fe0-40f4-81c0-a3915952426b/d4ff5ade-77fa-490a-a921-760304d03ec6"
           (reference "#PWR01") (unit 1)
-        )
-        (path "/e3b1e824-2fe0-40f4-81c0-a3915952426b/d4ff5ade-77fa-490a-a921-760304d03ec6"
-          (reference "#PWR01") (unit 1)
