File: kicad/epaper_board_layout.kicad_pcb (KiCad board)
At the start: 2 copper layers, 60 x 40 mm, 21 parts, among them J1 Conn_01x06_Pin, J2 Conn_01x06_Pin, J3 Conn_01x08_Pin, J4 Conn_01x02_Socket, Q1 PMOS - LP0701N3-G, SW1 SW_Push, U1 ATmega328-P, Y1 16Mhz

Commit message: Updated board schematic and layout because of FET labeled incorrectly in schematic.
Connections:
- Q1 pad 1: VCC -> VREF
- Q1 pad 3: VREF -> VCC
Other:
- board text added: "PRP"
Changed lines of the file:
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@@
     (pcbplotparams
       (layerselection 0x00010fc_ffffffff)
-      (plot_on_all_layers_selection 0x000d0f0_00000000)
-      (disableapertmacros false)
+      (plot_on_all_layers_selection 0x0000000_00000000)
+      (disableapertmacros true)
       (usegerberextensions true)
       (usegerberattributes true)
@@
     (property "Sheetname" "atmega328p")
     (property "Sim.Device" "PMOS")
-    (property "Sim.Pins" "1=D 2=G 3=S")
+    (property "Sim.Pins" "1=S 2=G 3=D")
     (property "Sim.Type" "VDMOS")
     (property "ki_description" "P-MOSFET transistor, drain/source/gate")
@@
       (stroke (width 0.1) (type solid)) (layer "F.Fab"))
     (pad "1" thru_hole rect (at 0 0 180) (size 1.3 1.3) (drill 0.75) (layers "*.Cu" "*.Mask")
-      (net 4 "VCC") (pinfunction "D") (pintype "passive"))
+      (net 13 "VREF") (pinfunction "D") (pintype "passive"))
     (pad "2" thru_hole circle (at 1.27 -1.27 180) (size 1.3 1.3) (drill 0.75) (layers "*.Cu" "*.Mask")
       (net 18 "Net-(Q1-G)") (pinfunction "G") (pintype "input"))
     (pad "3" thru_hole circle (at 2.54 0 180) (size 1.3 1.3) (drill 0.75) (layers "*.Cu" "*.Mask")
-      (net 13 "VREF") (pinfunction "S") (pintype "passive"))
+      (net 4 "VCC") (pinfunction "S") (pintype "passive"))
     (model "${KICAD6_3DMODEL_DIR}/Package_TO_SOT_THT.3dshapes/TO-92.wrl"
       (offset (xyz 0 0 0))
@@
   (gr_rect (start 100 100) (end 160 140)
     (stroke (width 0.0381) (type default)) (fill none) (layer "Edge.Cuts"))
-  (gr_text "BLK" (at 101.346 107.442) (layer "F.SilkS")
+  (gr_text "PRP" (at 101.346 107.442) (layer "F.SilkS")
     (effects (font (size 0.762 0.762) (thickness 0.127) bold) (justify left bottom))
   )
